File: Orders.sch (EAGLE design)
At the start: 0 parts

Commit message: Began BoM
Parts:
- added J1: 10104111-0001LF, USB:10104111-0001LF
- added JP1: (no value), pinhead:PINHD-1X4
- added R1, R2: (no value), rcl:R-EU_R1206
- added U$1: ATMEGA32U4-AU, adafruit:ATMEGA32U4-AU
Connections:
- new net +5V: J1.1, JP1.1
- new net D+: R2.2
- new net D-: R1.2
- new net GND: J1.5, J1.6, J1.7, J1.8, J1.9, JP1.2
- new net N$1: J1.2, R1.1
- new net N$2: J1.3, R2.1
- new net SCL: JP1.3
- new net SDA: JP1.4
Other:
- note added: "SCREEN"
- note added: "USB"
